File: OBJ_PCB_onju_by_imike78_2025-05-11.kicad_pcb (KiCad board)
At the start: 4 copper layers, 74.5 x 70.6 mm, 174 parts, among them J1 1775443-2, J2 usb_c, Q1 LBSS138WT1G, Q2 BC847B, SW1 CHS-01TA, U1 TPS62130, U10 SN74LVC125APWR, U11 MAX98357AETE_T, U12 FSUSB42MUX, U2 MIC5365-1.8YC5-TR, U3 TPS62130, U4 MIC5365-0.9YC5-TR, U5 ESP32-S3R8, U6 W25Q128JVSIQ, U7 XU316-1024-QF60B-C24, U8 W25Q128JVSIQ, U9 TLV73333PDBVR, Y1 40MHz, Y2 24MHz

Commit message: Add files via upload
Parts:
- added C77: 100nF, Capacitor_SMD:C_0603_1608Metric, F.Cu at (125.6, 106.1)
- added C78: 4.7uF, Capacitor_SMD:C_0603_1608Metric, F.Cu at (124.0, 106.1)
- added C79: 100nF, Capacitor_SMD:C_0603_1608Metric, F.Cu at (123.5, 111.2)
- added R22: 100k, Resistor_SMD:R_0402_1005Metric, F.Cu at (127.5, 107.0)
- added U13: AP22802AW5-7, Package_TO_SOT_SMD:SOT-23-5, F.Cu at (126.5, 109.6)
- moved R76 3.63 mm to (116.5, 109.3)
- moved U1 3.63 mm to (114.6, 105.6)
- moved C61 3.63 mm to (117.5, 105.8)
- moved C62 3.63 mm to (117.6, 108.3)
- moved C63 3.63 mm to (119.0, 105.8)
- moved C64 3.63 mm to (108.5, 105.1)
- moved C65 3.63 mm to (110.0, 100.3)
- moved C66 3.63 mm to (108.0, 100.4)
- moved L1 3.63 mm to (113.5, 100.8)
- moved R108 3.63 mm to (117.5, 102.8)
- moved R44 3.63 mm to (107.7, 102.8)
- moved R46 3.63 mm to (110.0, 105.0)
- moved R47 3.63 mm to (111.5, 105.0)
- moved R77 3.63 mm to (112.5, 109.8)
- renumbered POWER_IN to POWER_IN2

Commit message: Add files via upload
Parts:
- moved R5 13.9 mm to (149.8, 82.5), turned to 180 degrees
- moved C68 8.10 mm to (161.0, 76.5)
- moved D2 5.02 mm to (151.2, 81.2), turned to 180 degrees
- moved R4 3.62 mm to (163.0, 81.3), turned to 180 degrees
- moved C29 2.02 mm to (116.1, 66.2)
- moved R24 2.01 mm to (117.1, 66.2)
- moved R6 1.74 mm to (163.0, 80.0), turned to 180 degrees
- moved R25 1.26 mm to (115.1, 67.0)
- moved R26 1.26 mm to (114.1, 67.0)
- moved C14 1.01 mm to (118.6, 67.8)
- moved C15 1.01 mm to (120.6, 67.8)
- moved C18 1.01 mm to (121.1, 66.3)
- moved L5 1.01 mm to (120.1, 66.3)
- moved C16 1.01 mm to (118.1, 66.2)
- moved C17 1.01 mm to (119.1, 66.2)
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Routing:
- net GND: track 0.00 -> 44.9 mm
- net ESP_3V3: track 0.00 -> 19.8 mm, vias 0 -> 1
- net +5V: track 0.00 -> 19.4 mm
- net /XMOS/QSPI_CLK: track 0.00 -> 14.6 mm
- net /XMOS/QSPI_D0: track 0.00 -> 14.3 mm
- net /ESP32-S3R8/SPI_CS0: track 0.00 -> 12.9 mm
- net /ESP32-S3R8/SPI_Q: track 0.00 -> 12.7 mm
- net /XMOS/QSPI_D3: track 0.00 -> 12.6 mm, vias 0 -> 2
- net /ESP32-S3R8/SPI_WP: track 0.00 -> 12.3 mm, vias 0 -> 3
- net Net-(U5-XTAL_P): track 0.00 -> 10.5 mm
- net I2S_LRCK: track 0.00 -> 9.09 mm, vias 0 -> 2
- net /XMOS/QSPI_CS_N: track 0.00 -> 8.21 mm
- net VDD: track 0.00 -> 8.16 mm
- net VDDIO: track 0.00 -> 7.98 mm
- net I2S_BCLK: track 0.00 -> 7.07 mm, vias 0 -> 2
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
Commit message: Add files via upload
Parts:
- moved R2 4.11 mm to (132.5, 117.2), turned to 180 degrees
- moved R3 0.96 mm to (127.2, 121.5)
- moved D11 0.60 mm to (148.8, 108.0)
- moved D12 0.45 mm to (150.1, 107.4)
- turned C4 to -90 degrees
- turned R8 to -90 degrees
Routing:
- net +5V: track 19.4 -> 189.4 mm, vias 0 -> 7
- net GND: track 44.9 -> 183.7 mm, vias 0 -> 51
- net +3V3: track 0.00 -> 49.9 mm
- net ESP_USB_P: track 0.00 -> 43.0 mm, vias 0 -> 2
- net ESP_USB_N: track 0.00 -> 41.8 mm, vias 0 -> 2
- net VBUS: track 1.63 -> 38.6 mm, vias 0 -> 2
- net I2S2_DATA: track 0.00 -> 33.9 mm, vias 0 -> 2
- net I2C2_SDA: track 2.90 -> 36.8 mm, vias 0 -> 2
- net I2C2_SCL: track 2.62 -> 36.1 mm, vias 0 -> 2
- net ESP_MUTE_DET: track 1.26 -> 34.6 mm
- net /ESP32-S3R8/TOUCH_R: track 1.65 -> 31.1 mm
- net Net-(LED1-DOUT): track 0.00 -> 28.4 mm, vias 0 -> 2
- net +14V: track 0.00 -> 27.2 mm, vias 0 -> 2
- net ESP_WS2812: track 0.00 -> 22.8 mm
- net Net-(D10-A2): track 0.00 -> 20.9 mm, vias 0 -> 4
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- added copper zone on In2.Cu, net +0V9
- added copper zone on In2.Cu, net +1V8
- added copper zone on In2.Cu, net ESP_3V3
- added copper zone on In2.Cu, net VDD

Commit message: Github desktop implemented
Routing:
- net MUTE_ON: track 2.03 -> 11.4 mm
- net GND: track 183.7 -> 192.2 mm, vias 51 -> 55
- net VDDIO: track 7.98 -> 9.59 mm

Commit message: routing ongoing
Parts:
- moved C50 1.31 mm to (146.2, 70.4)
- moved R15 1.27 mm to (113.8, 69.2), turned to 0 degrees
- moved C53 0.64 mm to (144.0, 70.8)
- moved FB4 0.58 mm to (143.2, 75.5)
- moved R16 0.29 mm to (123.5, 74.0)
Routing:
- net I2S2_BCLK: track 0.00 -> 51.8 mm, vias 0 -> 1
- net I2S2_MCLK: track 0.00 -> 48.7 mm, vias 0 -> 3
- net I2C_SCL: track 4.68 -> 52.1 mm, vias 0 -> 2
- net I2C_SDA: track 4.03 -> 45.3 mm, vias 0 -> 2
- net XMOS_USB_P: track 0.00 -> 37.7 mm, vias 0 -> 2
- net XMOS_USB_N: track 0.00 -> 36.1 mm, vias 0 -> 2
- net ESP_IO40: track 0.00 -> 35.0 mm, vias 0 -> 2
- net I2S_DIN_SEC: track 0.00 -> 33.3 mm, vias 0 -> 2
- net +3V3: track 49.9 -> 82.0 mm
- net ESP_IO41: track 0.00 -> 31.3 mm, vias 0 -> 2
- net I2S_LRCK: track 9.09 -> 38.5 mm, vias 2 -> 3
- net MUTE_ON: track 11.4 -> 32.5 mm
- net GND: track 192.2 -> 200.5 mm, vias 55 -> 64
- net VDD: track 15.8 -> 20.3 mm
- net I2S_MCLK: track 0.00 -> 3.08 mm, vias 0 -> 1
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
Commit message: routing update
Routing:
- net /ESP32-S3R8/TOUCH_C: track 0.68 -> 80.1 mm
- net /ESP32-S3R8/TOUCH_L: track 1.04 -> 55.9 mm
- net I2S2_LRCLK: track 0.00 -> 39.9 mm, vias 0 -> 2
- net +5V: track 189.4 -> 197.5 mm, vias 7 -> 8
- net I2S_MCLK: track 3.08 -> 1.79 mm
- net I2S2_DATA: track 33.9 -> 35.0 mm
- net ESP_3V3: track 30.3 -> 30.4 mm, vias 10 -> 9

Commit message: routing update
Parts:
- removed R48, R49: 33R, Resistor_SMD:R_0402_1005Metric
- moved C35 0.58 mm to (102.5, 89.1)
Connections:
- U5 pad 52: GROVE_PWR -> unconnected-(U5-GPIO46-Pad52)
- U7 pad 33: /XMOS/XL_DN1 -> unconnected-(U7-X1D16-Pad33)
- U7 pad 35: /XMOS/XL_DN0 -> unconnected-(U7-X1D17-Pad35)
- U7 pad 36: Net-(U7-X1D18) -> unconnected-(U7-X1D18-Pad36)
- U7 pad 37: Net-(U7-X1D19) -> unconnected-(U7-X1D19-Pad37)
- U7 pad 48: XU316_WS2812 -> unconnected-(U7-X0D42-Pad48)
- U7 pad 50: BUT_A -> unconnected-(U7-X0D41-Pad50)
Routing:
- net /XMOS/MIC_CLK_M: track 2.31 -> 104.7 mm
- net +1V8: track 8.62 -> 53.3 mm, vias 0 -> 3
- net Net-(LED5-DOUT): track 0.00 -> 26.2 mm, vias 0 -> 4
- net +0V9: track 3.62 -> 29.7 mm, vias 0 -> 3
- net /XMOS/MIC_DATA_M: track 2.12 -> 22.8 mm, vias 0 -> 2
- net +3V3: track 82.0 -> 100.4 mm, vias 0 -> 6
- net /Power/USB_SEL: track 6.20 -> 13.1 mm
- net Net-(U7-X1D18): track 4.74 -> 0.00 mm
- net Net-(U7-X1D19): track 4.70 -> 0.00 mm
- net I2C2_SDA: track 36.4 -> 38.2 mm
- net GND: track 200.9 -> 202.5 mm, vias 64 -> 65
- net ESP_WS2812: track 22.8 -> 24.3 mm, vias 0 -> 2
- net +5V: track 197.5 -> 198.9 mm, vias 8 -> 10
- net MUTE_ON: track 32.5 -> 32.6 mm, vias 0 -> 2
- net Net-(LED2-DOUT): track 8.76 -> 8.75 mm, vias 0 -> 2

Commit message: routing update
Parts:
- moved R5 1.74 mm to (148.6, 81.2)
- moved C69 0.83 mm to (104.3, 86.2), turned to 45 degrees
- moved C63 0.76 mm to (119.8, 105.8)
- moved R1 0.59 mm to (130.6, 122.6)
- moved C4 0.44 mm to (123.3, 118.8)
- moved C61 0.26 mm to (117.8, 105.8)
- moved D3 0.22 mm to (102.9, 84.7)
- moved D5 0.14 mm to (106.3, 80.9)
- moved D7 0.10 mm to (166.1, 93.2)
- moved R8 0.10 mm to (125.0, 118.7)
- moved R7 0.05 mm to (123.2, 116.4)
Connections:
- J2 pad SH1: GND -> (no net)
- J2 pad SH2: GND -> (no net)
- J2 pad SH3: GND -> (no net)
- J2 pad SH4: GND -> (no net)
Routing:
- net VDD_MIC: track 10.8 -> 91.5 mm, vias 0 -> 2
- net /XMOS/MIC_DATA_M: track 22.8 -> 99.6 mm
- net ESP_3V3: track 30.4 -> 57.7 mm, vias 9 -> 10
- net +3V3: track 100.4 -> 123.9 mm
- net VDDIO: track 9.59 -> 27.3 mm
- net VDD: track 20.3 -> 27.9 mm, vias 0 -> 7
- net GND: track 202.5 -> 197.3 mm, vias 65 -> 58
- net Net-(D10-A2): track 20.9 -> 24.9 mm
- net +14V: track 27.2 -> 30.3 mm
- net Net-(C4-Pad1): track 2.98 -> 3.95 mm
- net ESP_WS2812: track 24.3 -> 25.2 mm
- net Net-(LED1-DOUT): track 28.3 -> 27.6 mm
- net +5V: track 198.9 -> 199.6 mm
- net Net-(U3-FB): track 11.0 -> 11.5 mm
- net /ESP32-S3R8/SPI_WP: vias 3 -> 2
- added copper zone on F.Cu, net GND
- added copper zone on In1.Cu, net GND
