File: nest-mini-v2-drop-in-pcb.kicad_pcb (KiCad board)
At the start: 4 copper layers, 74.5 x 70.6 mm, 180 parts, among them J1 1775443-2, J2 usb_c, Q1 LBSS138WT1G, Q2 BC847B, SW1 SMXS_01K_TP, U1 TPS62130, U10 SN74LVC125APWR, U11 MAX98357AETE_T, U12 FSUSB42MUX, U13 AP22802AW5-7, U2 MIC5365-1.8YC5-TR, U3 TPS62130, U4 TPS7A0309PDBVR, U5 ESP32-S3R8, U6 W25Q128JVSIQ, U7 XU316-1024-QF60B-C24, U8 W25Q128JVSIQ, U9 TLV73333PDBVR, Y1 40MHz, Y2 24MHz

Commit message: rev2 update
Connections:
- U5 pad 23: AUDIO_DET -> ESP_MUTE_DET
- U5 pad 38: ESP_MUTE_DET -> unconnected-(U5-GPIO33-Pad38)
- U5 pad 39: X316_RST -> unconnected-(U5-GPIO34-Pad39)
- U5 pad 51: WS2812_PWR -> X316_RST
Routing:
- net ESP_MUTE_DET: track 34.6 -> 40.2 mm, vias 0 -> 2
Changed lines of the file:
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@@
 	(net 55 "unconnected-(U5-GPIO37-Pad42)")
 	(net 56 "I2C2_SCL")
-	(net 57 "AUDIO_DET")
+	(net 57 "unconnected-(U5-GPIO33-Pad38)")
 	(net 58 "I2S2_DATA")
 	(net 59 "ESP_USB_P")
@@
 	(net 64 "/ESP32-S3R8/SPI_CS0")
 	(net 65 "AUDIO_PA_EN")
-	(net 66 "WS2812_PWR")
+	(net 66 "unconnected-(U5-GPIO34-Pad39)")
 	(net 67 "unconnected-(U5-GPIO1-Pad6)")
 	(net 68 "ESP_IO48")
@@
 			)
 		)
+		(model "${KIPRJMOD}/parts/QFN_F60B-C24_XMO.step"
+			(offset
+				(xyz 0 0 0)
+			)
+			(scale
+				(xyz 1 1 1)
+			)
+			(rotate
+				(xyz 0 0 0)
+			)
+		)
 	)
 	(footprint "Crystal:Crystal_SMD_3225-4Pin_3.2x2.5mm"
@@
 		(at 118.060362 73.930999 -90)
 		(property "Reference" "U5"
-			(at 4.84 -2.54 180)
+			(at 4.84 -2.54 0)
 			(layer "F.SilkS")
 			(effects
@@
 			(layers "F.Cu" "F.Mask" "F.Paste")
 			(roundrect_rratio 0.125)
-			(net 57 "AUDIO_DET")
+			(net 60 "ESP_MUTE_DET")
 			(pinfunction "GPIO17")
 			(pintype "bidirectional")
@@
 			(layers "F.Cu" "F.Mask" "F.Paste")
 			(roundrect_rratio 0.125)
-			(net 60 "ESP_MUTE_DET")
+			(net 57 "unconnected-(U5-GPIO33-Pad38)")
 			(pinfunction "GPIO33")
-			(pintype "bidirectional")
+			(pintype "bidirectional+no_connect")
 			(solder_mask_margin 0.102)
 		)
@@
 			(layers "F.Cu" "F.Mask" "F.Paste")
 			(roundrect_rratio 0.125)
-			(net 61 "X316_RST")
+			(net 66 "unconnected-(U5-GPIO34-Pad39)")
 			(pinfunction "GPIO34")
-			(pintype "bidirectional")
+			(pintype "bidirectional+no_connect")
 			(solder_mask_margin 0.102)
 		)
@@
 			(layers "F.Cu" "F.Mask" "F.Paste")
 			(roundrect_rratio 0.125)
-			(net 66 "WS2812_PWR")
+			(net 61 "X316_RST")
 			(pinfunction "GPIO45")
 			(pintype "bidirectional")
@@
 			)
 		)
+		(model "${KIPRJMOD}/parts/ESP32-S3R8.step"
+			(offset
+				(xyz 0 0 0)
+			)
+			(scale
+				(xyz 1 1 1)
+			)
+			(rotate
+				(xyz -90 -0 -0)
+			)
+		)
 	)
 	(footprint "Resistor_SMD:R_0402_1005Metric"
@@
 			)
 		)
+		(model "${KIPRJMOD}/parts/SN74LVC125APWR.step"
+			(offset
+				(xyz 0 0 0)
+			)
+			(scale
+				(xyz 1 1 1)
+			)
+			(rotate
+				(xyz -90 -0 -0)
+			)
+		)
 	)
 	(footprint "Onju:MIC_T3902"
@@
 		)
 		(embedded_fonts no)
-		(model "D:/temp/Onju voice/Parts/DMM-3526-B-R.step"
+		(model "${KIPRJMOD}/parts/DMM-3526-B-R.step"
 			(offset
-				(xyz 0 0 0.4)
+				(xyz 0 0 0.45)
 			)
 			(scale
@@
 			)
 		)
+		(model "${KIPRJMOD}/parts/DMM-3526-B-R.step"
+			(offset
+				(xyz 0 0 0.45)
+			)
+			(scale
+				(xyz 1 1 1)
+			)
+			(rotate
+				(xyz -90 -0 -0)
+			)
+		)
 	)
 	(footprint "Diode_SMD:D_0402_1005Metric"
@@
 	)
 	(segment
+		(start 115.430999 74.530999)
+		(end 115.5 74.6)
+		(width 0.15)
+		(layer "F.Cu")
+		(net 60)
+	)
+	(segment
 		(start 147.785 78.75)
 		(end 150.285 81.25)
@@
 	)
 	(segment
-		(start 119.060362 77.375999)
-		(end 119.060362 78.310362)
-		(width 0.15)
-		(layer "F.Cu")
-		(net 60)
-	)
-	(segment
 		(start 119.25 78.5)
 		(end 123.5 78.5)
@@
 	)
 	(segment
-		(start 119.060362 78.310362)
-		(end 119.25 78.5)
+		(start 114.615362 74.530999)
+		(end 115.430999 74.530999)
+		(width 0.15)
+		(layer "F.Cu")
+		(net 60)
+	)
+	(segment
+		(start 119.25 78.5)
+		(end 119.2 78.5)
 		(width 0.15)
 		(layer "F.Cu")
 		(net 60)
 	)
+	(via
+		(at 115.5 74.6)
+		(size 0.4)
+		(drill 0.2)
+		(layers "F.Cu" "B.Cu")
+		(net 60)
+	)
+	(via
+		(at 119.2 78.5)
+		(size 0.4)
+		(drill 0.2)
+		(layers "F.Cu" "B.Cu")
+		(net 60)
+	)
+	(segment
+		(start 117 77)
+		(end 118.5 78.5)
+		(width 0.15)
+		(layer "In2.Cu")
+		(net 60)
+	)
+	(segment
+		(start 117 76.1)
+		(end 117 77)
+		(width 0.15)
+		(layer "In2.Cu")
+		(net 60)
+	)
+	(segment
+		(start 118.5 78.5)
+		(end 119.2 78.5)
+		(width 0.15)
+		(layer "In2.Cu")
+		(net 60)
+	)
+	(segment
+		(start 115.5 74.6)
+		(end 117 76.1)
+		(width 0.15)
+		(layer "In2.Cu")
+		(net 60)
+	)
