File: nest-mini-v2-drop-in-pcb.kicad_pcb (KiCad board)
At the start: 4 copper layers, 74.5 x 70.6 mm, 185 parts, among them J1 1775443-2, J2 usb_c, Q1 LBSS138WT1G, Q2 BC847B, Q3 LBSS138WT1G, SW1 SMXS_01K_TP, U1 TPS62130, U10 SN74LVC125APWR, U11 MAX98357AETE_T, U12 FSUSB42MUX, U13 AP22802AW5-7, U2 MIC5365-1.8YC5-TR, U3 TPS62130, U4 TPS7A0309PDBVR, U5 ESP32-S3R8, U6 W25Q128JVSIQ, U7 XU316-1024-QF60B-C24, U8 W25Q128JVSIQ, U9 TLV73333PDBVR, Y1 40MHz, Y2 24MHz

Commit message: rev2 update
Parts:
- removed TP1: BOOT, TestPoint:TestPoint_Pad_D1.0mm
- removed TP2: GND, TestPoint:TestPoint_Pad_D1.0mm
- removed TP3: RESET, TestPoint:TestPoint_Pad_D1.0mm
- added SW2: BOOT, Onju:SW-SMD_4P-L4.2-W3.2-P2.15-LS4.5, F.Cu at (137.5, 80.8)
- added SW3: Reset, Onju:SW-SMD_4P-L4.2-W3.2-P2.15-LS4.5, F.Cu at (119.6, 90.5)
Routing:
- net ESP_RST: track 17.9 -> 29.2 mm
- net ESP_BOOT: track 9.77 -> 5.55 mm
- net GND: track 198.6 -> 195.0 mm, vias 315 -> 313

Commit message: rev2 update
Routing:
- net ESP_BOOT: track 5.55 -> 30.6 mm, vias 0 -> 2
Changed lines of the file:
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@@
 	)
 	(segment
-		(start 129.450999 122.950999)
+		(start 128.7 122.2)
 		(end 128 121.5)
 		(width 0.25)
@@
 	)
 	(segment
-		(start 135.049001 122.950999)
-		(end 129.450999 122.950999)
+		(start 135 122.2)
+		(end 128.7 122.2)
 		(width 0.25)
 		(layer "In2.Cu")
@@
 	(segment
 		(start 135.4 122.6)
-		(end 135.049001 122.950999)
+		(end 135 122.2)
 		(width 0.25)
 		(layer "In2.Cu")
@@
 	)
 	(segment
+		(start 135.248607 79.5)
+		(end 135.506849 79.758242)
+		(width 0.15)
+		(layer "F.Cu")
+		(net 32)
+	)
+	(segment
+		(start 119.060362 71.260362)
+		(end 119.1 71.3)
+		(width 0.15)
+		(layer "F.Cu")
+		(net 32)
+	)
+	(segment
+		(start 132.7 79.5)
+		(end 135.248607 79.5)
+		(width 0.15)
+		(layer "F.Cu")
+		(net 32)
+	)
+	(segment
 		(start 117.100362 66.76)
 		(end 117.100362 67.852388)
@@
 	)
 	(segment
+		(start 119.060362 70.485999)
+		(end 119.060362 71.260362)
+		(width 0.15)
+		(layer "F.Cu")
+		(net 32)
+	)
+	(segment
 		(start 117.070362 66.73)
 		(end 117.100362 66.76)
@@
 		(net 32)
 	)
+	(via
+		(at 132.7 79.5)
+		(size 0.4)
+		(drill 0.2)
+		(layers "F.Cu" "B.Cu")
+		(net 32)
+	)
+	(via
+		(at 119.1 71.3)
+		(size 0.4)
+		(drill 0.2)
+		(layers "F.Cu" "B.Cu")
+		(net 32)
+	)
+	(segment
+		(start 119.1 71.3)
+		(end 120.8 69.6)
+		(width 0.15)
+		(layer "In2.Cu")
+		(net 32)
+	)
+	(segment
+		(start 120.8 69.6)
+		(end 127.7 69.6)
+		(width 0.15)
+		(layer "In2.Cu")
+		(net 32)
+	)
+	(segment
+		(start 132.7 74.6)
+		(end 132.7 79.5)
+		(width 0.15)
+		(layer "In2.Cu")
+		(net 32)
+	)
+	(segment
+		(start 127.7 69.6)
+		(end 132.7 74.6)
+		(width 0.15)
+		(layer "In2.Cu")
+		(net 32)
+	)

Commit message: rev2 update
Parts:
- R33: value 470K -> 470k
- R34: value 10K -> 10k
Changed lines of the file:
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@@
 			)
 		)
+		(property "Function" "ESP32"
+			(at 0 0 270)
+			(unlocked yes)
+			(layer "F.Fab")
+			(hide yes)
+			(effects
+				(font
+					(size 1 1)
+					(thickness 0.15)
+				)
+			)
+		)
+		(property "Manufacturer" "C&K"
+			(at 0 0 270)
+			(unlocked yes)
+			(layer "F.Fab")
+			(hide yes)
+			(effects
+				(font
+					(size 1 1)
+					(thickness 0.15)
+				)
+			)
+		)
+		(property "Manufacturer Part" "PTS810SJS250SMTRLFS"
+			(at 0 0 270)
+			(unlocked yes)
+			(layer "F.Fab")
+			(hide yes)
+			(effects
+				(font
+					(size 1 1)
+					(thickness 0.15)
+				)
+			)
+		)
+		(property "Supplier Part" "C221897"
+			(at 0 0 270)
+			(unlocked yes)
+			(layer "F.Fab")
+			(hide yes)
+			(effects
+				(font
+					(size 1 1)
+					(thickness 0.15)
+				)
+			)
+		)
+		(property "LCSC Part #" "C221897"
+			(at 0 0 270)
+			(unlocked yes)
+			(layer "F.Fab")
+			(hide yes)
+			(effects
+				(font
+					(size 1 1)
+					(thickness 0.15)
+				)
+			)
+		)
 		(sheetname "/ESP32-S3R8/")
 		(sheetfile "esp32.kicad_sch")
@@
 			)
 		)
-		(property "Value" "470K"
+		(property "Value" "470k"
 			(at 0 1.17 90)
 			(layer "F.Fab")
@@
 			)
 		)
+		(property "LCSC Part #" "C25790"
+			(at 0 0 90)
+			(unlocked yes)
+			(layer "F.Fab")
+			(hide yes)
+			(effects
+				(font
+					(size 1 1)
+					(thickness 0.15)
+				)
+			)
+		)
 		(property ki_fp_filters "Resistor:R0402")
 		(sheetname "/XMOS/")
@@
 			)
 		)
-		(property "Supplier Part" "C27124"
+		(property "Supplier Part" "C16526"
 			(at 0 0 270)
 			(unlocked yes)
@@
 			)
 		)
+		(property "Function" "ESP32"
+			(at 0 0 0)
+			(unlocked yes)
+			(layer "F.Fab")
+			(hide yes)
+			(effects
+				(font
+					(size 1 1)
+					(thickness 0.15)
+				)
+			)
+		)
+		(property "Manufacturer" "C&K"
+			(at 0 0 0)
+			(unlocked yes)
+			(layer "F.Fab")
+			(hide yes)
+			(effects
+				(font
+					(size 1 1)
+					(thickness 0.15)
+				)
+			)
+		)
+		(property "Manufacturer Part" "PTS810SJS250SMTRLFS"
+			(at 0 0 0)
+			(unlocked yes)
+			(layer "F.Fab")
+			(hide yes)
+			(effects
+				(font
+					(size 1 1)
+					(thickness 0.15)
+				)
+			)
+		)
+		(property "Supplier Part" "C221897"
+			(at 0 0 0)
+			(unlocked yes)
+			(layer "F.Fab")
+			(hide yes)
+			(effects
+				(font
+					(size 1 1)
+					(thickness 0.15)
+				)
+			)
+		)
+		(property "LCSC Part #" "C221897"
+			(at 0 0 0)
+			(unlocked yes)
+			(layer "F.Fab")
+			(hide yes)
+			(effects
+				(font
+					(size 1 1)
+					(thickness 0.15)
+				)
+			)
+		)
 		(sheetname "/ESP32-S3R8/")
 		(sheetfile "esp32.kicad_sch")
@@
 			)
 		)
+		(property "LCSC Part #" "C25076"
+			(at 0 0 270)
+			(unlocked yes)
+			(layer "F.Fab")
+			(hide yes)
+			(effects
+				(font
+					(size 1 1)
+					(thickness 0.15)
+				)
+			)
+		)
 		(sheetname "/XMOS/")
 		(sheetfile "xmos.kicad_sch")
@@
 			)
 		)
+		(property "LCSC Part #" "C383201"
+			(at 0 0 0)
+			(unlocked yes)
+			(layer "F.Fab")
+			(hide yes)
+			(effects
+				(font
+					(size 1 1)
+					(thickness 0.15)
+				)
+			)
+		)
 		(sheetname "/XMOS/")
 		(sheetfile "xmos.kicad_sch")
@@
 			)
 		)
-		(property "Value" "10K"
+		(property "Value" "10k"
 			(at 0 1.17 270)
 			(layer "F.Fab")
@@
 			)
 		)
+		(property "LCSC Part #" "C25744"
+			(at 0 0 270)
+			(unlocked yes)
+			(layer "F.Fab")
+			(hide yes)
+			(effects
+				(font
+					(size 1 1)
+					(thickness 0.15)
+				)
+			)
+		)
 		(sheetname "/XMOS/")
 		(sheetfile "xmos.kicad_sch")
@@
 			(at 0 0 270)
 			(unlocked yes)
+			(layer "F.Fab")
+			(hide yes)
+			(effects
+				(font
+					(size 1 1)
+					(thickness 0.15)
+				)
+			)
+		)
+		(property "LCSC Part #" "C1525"
+			(at 0 0 270)
+			(unlocked yes)

Commit message: rev2 update
Parts:
- moved C51 0.25 mm to (151.1, 66.7)
Connections:
- U7 pad 33: unconnected-(U7-X1D16-Pad33) -> /XMOS/XL_DN1
- U7 pad 35: unconnected-(U7-X1D17-Pad35) -> /XMOS/XL_DN0
Routing:
- net GND: track 195.0 -> 192.5 mm, vias 313 -> 301
- net I2C2_SCL: track 38.4 -> 36.7 mm

Commit message: update for production
Parts:
- U8: value W25Q128JVSIQ -> W25Q32JVSSIQ
Connections:
- U5 pad 22: ECO_A -> unconnected-(U5-XTAL_32K_N-Pad22)
- U5 pad 24: ECO_B -> unconnected-(U5-GPIO18-Pad24)
- U5 pad 36: ESP_IO48 -> unconnected-(U5-SPICLK_N-Pad36)
- U7 pad 18: /XMOS/TDI -> unconnected-(U7-TDI-Pad18)
- U7 pad 20: /XMOS/TDO -> unconnected-(U7-TDO-Pad20)
- U7 pad 23: /XMOS/TMS -> unconnected-(U7-TMS-Pad23)
- U7 pad 24: /XMOS/TCK -> unconnected-(U7-TCK-Pad24)
- U7 pad 33: /XMOS/XL_DN1 -> unconnected-(U7-X1D16-Pad33)
- U7 pad 35: /XMOS/XL_DN0 -> unconnected-(U7-X1D17-Pad35)
- U7 pad 46: /XMOS/XMOS_MUTE_DET -> unconnected-(U7-X0D40-Pad46)
- U7 pad 51: ESP_IO40 -> unconnected-(U7-X0D43-Pad51)
- U7 pad 55: /XMOS/XOD31 -> unconnected-(U7-X0D31-Pad55)
- U7 pad 56: RST_DAC -> unconnected-(U7-X0D32-Pad56)
- U7 pad 58: ESP_IO41 -> unconnected-(U7-X0D33-Pad58)
Routing:
- net ESP_IO40: track 33.9 -> 0.00 mm, vias 2 -> 0
- net ESP_IO41: track 31.3 -> 0.00 mm, vias 2 -> 0
- net GND: track 192.5 -> 178.5 mm, vias 301 -> 359
- net ESP_RST: track 29.2 -> 28.3 mm
