File: nest-mini-v2-drop-in-pcb.kicad_pcb (KiCad board)
At the start: 4 copper layers, 74.5 x 70.6 mm, 238 parts, among them J1 usb_c, J2 Conn_01x05, J3 XTAG DEV, J4 XMOS JTAG, J5 1775443-2, Q1 LBSS138WT1G, Q2 LBSS138WT1G, Q3 BC847B, SW1 Reset, SW2 BOOT, U1 CUS-12TB, U10 XU316-1024-QF60B-C24​, U11 W25Q32JVSSIQ, U12 SN74LVC125APWR, U13 TLV73333PDBVR, U14 TAS5805MPWPR, U15 MPR121QR2, U2 TS3USB221ERSER, U3 TPS62130, U4 AP22802AW5-7, U5 MIC5365-1.8YC5-TR, U6 TPS7A0309PDBVR, U7 TPS62130, U8 ESP32-S3R8, U9 W25Q128JVSIQ, X1 24MHz 12pF, Y1 40MHz

Commit message: adding esp32c6 for OTBR
Parts:
- moved R67 4.10 mm to (129.0, 99.4)
- moved C98 0.38 mm to (139.7, 82.7)
- moved R72 0.38 mm to (139.7, 81.7)
Routing:
- net /XMOS/MIC_DATA_M_2: track 1.00 -> 56.9 mm, vias 0 -> 3
- net /XMOS/MIC_CLK_M: track 76.0 -> 124.8 mm, vias 2 -> 3
- net Net-(U15-ELEC1): track 0.00 -> 41.8 mm, vias 0 -> 2
- net /ESP32-S3R8/TOUCH_IRQ: track 0.00 -> 30.7 mm, vias 0 -> 1
- net VDD_MIC: track 87.4 -> 117.9 mm, vias 2 -> 3
- net DVDD: track 8.61 -> 4.33 mm
- net +3V3: track 98.0 -> 102.1 mm, vias 13 -> 14
- net XU316_RST: track 11.9 -> 8.32 mm
- net I2C_SCL: track 80.6 -> 79.2 mm
- net I2C_SDA: track 80.7 -> 79.5 mm
- net GND: vias 173 -> 207

Commit message: WiP update
Parts:
- added AE2: 2450AT18A100E, RF_Antenna:Johanson_2450AT18x100, F.Cu at (200.0, 84.2)
- added C100: 1.2pF, Capacitor_SMD:C_0402_1005Metric, F.Cu at (190.8, 71.6)
- added C101: 12pF, Capacitor_SMD:C_0402_1005Metric, F.Cu at (190.8, 73.6)
- added C102: 12pF, Capacitor_SMD:C_0402_1005Metric, F.Cu at (190.8, 75.5)
- added C103: 1uF, Capacitor_SMD:C_0402_1005Metric, F.Cu at (190.8, 77.5)
- added C104: 12pF, Capacitor_SMD:C_0402_1005Metric, F.Cu at (190.8, 79.5)
- added C105: 1uF, Capacitor_SMD:C_0402_1005Metric, F.Cu at (190.8, 81.5)
- added C106: 100nF, Capacitor_SMD:C_0402_1005Metric, F.Cu at (193.6, 71.6)
- added C107: 12pF, Capacitor_SMD:C_0402_1005Metric, F.Cu at (193.6, 73.6)
- added C108: 2.4pF, Capacitor_SMD:C_0402_1005Metric, F.Cu at (193.6, 75.5)
- added C109: 100nF, Capacitor_SMD:C_0402_1005Metric, F.Cu at (193.6, 77.5)
- added C110: 100nF, Capacitor_SMD:C_0402_1005Metric, F.Cu at (193.6, 79.5)
- added C111: 1uF, Capacitor_SMD:C_0402_1005Metric, F.Cu at (193.6, 81.5)
- added C112: 10uF, Capacitor_SMD:C_0402_1005Metric, F.Cu at (196.5, 71.6)
- added C113: 100nF, Capacitor_SMD:C_0402_1005Metric, F.Cu at (196.5, 73.6)
- added C114: 100nF, Capacitor_SMD:C_0402_1005Metric, F.Cu at (196.5, 75.5)
- added C115: 100nF, Capacitor_SMD:C_0603_1608Metric, F.Cu at (199.9, 74.4)
- added D7: LRB520S-30T1G, Diode_SMD:D_SOD-523, F.Cu at (199.7, 76.9)
- added FB6: 120R, Onju:BLM18PG121SN1D, F.Cu at (199.9, 71.9)
- added L10: 24nH, Inductor_SMD:L_0402_1005Metric, F.Cu at (187.9, 75.6)
- added L11: 2.2nH, Inductor_SMD:L_0402_1005Metric, F.Cu at (187.9, 77.6)
- added L8: 3.3nH, Inductor_SMD:L_0402_1005Metric, F.Cu at (187.9, 71.6)
- added L9: 2.7nH, Inductor_SMD:L_0402_1005Metric, F.Cu at (187.9, 73.6)
- added R74: 10k, Resistor_SMD:R_0402_1005Metric, F.Cu at (187.9, 79.6)
- added R75: 10k, Resistor_SMD:R_0402_1005Metric, F.Cu at (187.9, 81.6)
- added R76: 10k, Resistor_SMD:R_0402_1005Metric, F.Cu at (187.9, 83.6)
- added R77: 10k, Resistor_SMD:R_0402_1005Metric, F.Cu at (187.9, 85.5)
- added TP14: TOUCH_R, Onju:Touchpad, B.Cu at (162.8, 89.1)
- added TP15: TOUCH_C, Onju:Touchpad, B.Cu at (135.9, 115.9)
- added TP16: TOUCH_L, Onju:Touchpad, B.Cu at (108.8, 89.1)
- added U16: ESP32-C6FH8, Onju:ESP32-C6FH4, F.Cu at (193.5, 86.1)
- added Y2: 40MHz, Crystal:Crystal_SMD_2016-4Pin_2.0x1.6mm, F.Cu at (199.2, 87.7)
- moved R69 0.30 mm to (131.8, 112.1)
- renumbered U1 to SW3
Connections:
- net ESP_USB_N renamed S3_USB_N
- net ESP_USB_P renamed S3_USB_P
- J1 pad 0: (no net) -> GND
- U2 pad 3: XMOS_USB_P -> C6_USB_P
- U2 pad 4: XMOS_USB_N -> C6_USB_N
Routing:
- net XMOS_USB_P: track 28.2 -> 0.00 mm
- net XMOS_USB_N: track 27.4 -> 0.00 mm
- net Net-(LED1-DOUT): track 29.3 -> 30.4 mm
- net VDD_MIC: track 117.9 -> 118.7 mm
- net GND: vias 207 -> 213
