File: nest-mini-v2-drop-in-pcb.kicad_sch (KiCad schematic)
At the start: 0 parts

Commit message: complete redesign
Other:
- title: Nest mini drop in PCB replacement -> Drop in replacement PCB for Nest mini GEN2
Changed lines of the file:
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@@
 	(paper "A4")
 	(title_block
-		(title "Nest mini drop in PCB replacement")
+		(title "Drop in replacement PCB for Nest mini GEN2")
 		(rev "v1")
 		(company "by iMike78 (inpired by Onju voice and HA VPE)")
