File: xmos.kicad_sch (KiCad schematic)
At the start: 82 parts, among them J3 XTAG DEV, J4 XMOS JTAG, Q1 LBSS138WT1G, Q2 LBSS138WT1G, Q3 BC847B, U10 SN74LVC125APWR, U11 TLV73333PDBVR, U8 XU316-1024-QF60B-C24​, U9 W25Q32JVSSIQ, X1 24MHz 12pF

Commit message: v2 hardware revision
MPR121 touch controller added to replace the esp32-s3 internal touch interface
Parts:
- added TP11: XU316_RST, TestPoint:TestPoint_Pad_D1.0mm, symbol Connector:TestPoint
- added TP12: MUTE, TestPoint:TestPoint_Pad_D1.0mm, symbol Connector:TestPoint
- renumbered C40 to C42, C41 to C43, C42 to C44, C43 to C45, C44 to C46, C45 to C47, C46 to C48, C47 to C49, C48 to C50, C49 to C51, C50 to C52, C51 to C53, C52 to C54, C53 to C55, C54 to C56, C55 to C57, C56 to C58, C57 to C59, C58 to C60, C63 to C62, C64 to C63, C65 to C64, C66 to C65, C67 to C66, C68 to C67, C69 to C68, C70 to C69, C71 to C70, C72 to C71, C73 to C72, C92 to C73, D5 to D6, R30 to R34, R31 to R35, R32 to R36, R33 to R37, R34 to R38, R35 to R39, R37 to R40, R45 to R42, R48 to R43, R49 to R44, R69 to R45, R70 to R46, R51 to R47, R52 to R48, R53 to R49, R54 to R50, R44 to R51, R55 to R52, R56 to R53, R57 to R54, R58 to R55, R59 to R56, R60 to R57, R61 to R58, R62 to R59, R63 to R60, R42 to R61, R64 to R62, R65 to R63, R43 to R64, R66 to R65, TP4 to TP10, U8 to U10, U9 to U11, U10 to U12, U11 to U13
Connections:
- net MUTE: now also TP12.1
- net XU316_RST: now also TP11.1
- net XMOS_USB_N: now reaches U10.28 (USB_DM)
- net XMOS_USB_P: now reaches U10.29 (USB_DP)
- no-connect marks 12 -> 10
Other:
- moved on the sheet: C67, R55, R57
