File: audio.kicad_sch (KiCad schematic)
At the start: 29 parts, among them J5 1775443-2, U14 TAS5805MPWPR

Commit message: Publish KiCad 10 hardware updates
Refresh the Nest Mini v2 drop-in PCB project in KiCad 10 and publish the accumulated schematic and board updates as a single clean mainline change.

Remove the unused USB-C power/input branch from the power sheet, including the USB connector path, data switching, VBUS switching, and associated support parts, while preserving the pogo-accessible USB signals where needed. Add the ESP32-C6 1x05 pogo connector with the J2-style pin order for GND, boot, reset, USB D-, and USB D+ without a 3.3 V pin.

Add a 5 V SN74AHCT1G125 buffer for the LED data input, with local decoupling and a 47 ohm series output resistor, so the LED chain receives a buffered LED_WS2812_5V signal from the ESP_WS2812 control net.

Carry forward the KiCad 10 project save state and schematic cleanups for the XMOS, ESP32, audio, LED, and power sheets without changing the TAS amplifier topology.
Parts:
- R69: renamed from R68; now not fitted
- R70: renamed from R69; MPN 0402WGF0000TCE -> ERJ-6GEY0R00V; Manufacturer UNI-ROYAL(Uniroyal Elec) -> Panasonic Industry; Manufacturer Part 0402WGF0000TCE -> ERJ-6GEY0R00V
- renumbered C86 to C100, C87 to C101, C88 to C102, C89 to C103, C90 to C104, C91 to C105, C74 to C88, C75 to C89, C76 to C90, C77 to C91, C78 to C92, C79 to C93, C80 to C94, C81 to C95, C82 to C96, C83 to C97, C84 to C98, C85 to C99, L6 to L11, L7 to L12, R66 to R67, R67 to R68, R70 to R71, R71 to R72, TP13 to TP11, U14 to U13
