File: audio.kicad_sch (KiCad schematic)
At the start: 29 parts, among them J5 1775443-2, U13 TAS5805MPWPR

Commit message: Publish ESP32-P4 multi-sheet hardware redesign
Parts:
- removed R69: 0R, Resistor_SMD:R_0805_2012Metric, symbol Seeed_libdb:Resistors/301010000
- C92: Function MIC -> TAS
- J5: Function AUDIO -> TAS
- R70, R71, U13: Function (none) -> TAS
- R72: Function XMOS -> TAS
Connections:
- net SDOUT: now reaches U13.9 (SDOUT)
- no-connect marks 1 -> 0

Commit message: v3 hardware changes
Full redesing, ready for prototype order
Parts:
- added D6: SMAJ15A, Diode_SMD:D_SMA, symbol Diode:SMAJ15A
- added TP1: max +15V!, TestPoint:TestPoint_THTPad_D3.0mm_Drill1.5mm, symbol Connector:TestPoint
- added TP8, TP9: SP OUT, TestPoint:TestPoint_Pad_D2.0mm, symbol Connector:TestPoint
- C92: value 100nF -> 1uF; LCSC Part # C1525 -> (none); Manufacturer Part CL05B104KO5NNNC -> (none); Supplier Part C1525 -> (none)
- L11, L12: footprint Onju:XAL4040-103MEC -> Inductor_SMD:L_Coilcraft_XAL5050-XXX; Current 3A -> 4.9A; DCR 84 mOhm -> 41 mOhm; Manufacturer (none) -> Coilcraft; Manufacturer Part (none) -> XAL5050-103MEC
- R71: value 0R -> 4.7k
- TP11: value TestPoint -> PA_EN
Connections:
- net +14V: now also D6.1 (A1), TP1.1
- net DGND: no longer R71.1
- net DVDD: now also R71.1
- net GND: now also D6.2 (A2)
- net at C100.1, J5.1, L11.2: now also TP8.1
- net at C101.1, J5.2, L12.2: now also TP9.1
Other:
- moved on the sheet: C100, C101, C102, C103, C104, C105, C88, C89, C90, C91, C92, C93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

Commit message: v3 hardware ready for prototyping
Parts:
- C100, C101: LCSC Part # (none) -> C472832; Manufacturer MuRata -> Samsung Electro-Mechanics; Manufacturer Part GRM188R72A10 -> CL21B684KBFVPNE; Supplier Part (none) -> C472832; Voltage 100V -> 50V
- C104, C94: LCSC Part # (none) -> C19666; Manufacturer (none) -> Samsung Electro-Mechanics; Manufacturer Part (none) -> CL10A475KO8NNNC; Supplier Part (none) -> C19666; Voltage 10V -> 16V
- C105, C96: LCSC Part # (none) -> C14663; Manufacturer (none) -> YAGEO; Manufacturer Part (none) -> CC0603KRX7R9BB104; Supplier Part (none) -> C14663; Voltage 16V -> 50V
- C88, C89, C90, C91: LCSC Part # (none) -> C21120; Manufacturer (none) -> Samsung Electro-Mechanics; Manufacturer Part (none) -> CL10B224KA8NNNC; Supplier Part (none) -> C21120; Voltage 50V -> 25V
- C92: Dielectric X7R -> X5R; LCSC Part # (none) -> C52923; Manufacturer Part (none) -> CL05A105KA5NQNC; Supplier Part (none) -> C52923; Voltage 16V -> 25V
- C93, C95, C98, C99: LCSC Part # C86816 -> C45783; Manufacturer Murata Electronics -> Samsung Electro-Mechanics; Manufacturer Part GRM21BR61E226ME44L -> CL21A226MAQNNNE; Supplier Part C86816 -> C45783
- D6: Function (none) -> POWER; LCSC Part # (none) -> C148216; Manufacturer (none) -> Littelfuse; Manufacturer Part (none) -> SMAJ15A; Supplier Part (none) -> C148216
- J5: MP 1775443-2 -> 5-1775443-2; Manufacturer Part 1775443-2 -> 5-1775443-2
- L11, L12: LCSC Part # (none) -> C5441578; Supplier Part (none) -> C5441578
- R67: Function (none) -> TAS; LCSC Part # (none) -> C17888; Manufacturer (none) -> UNI-ROYAL(Uniroyal Elec); Manufacturer Part (none) -> 1206W4F0000T5E; Supplier Part (none) -> C17888
- R68: Function (none) -> ESP32-P4; LCSC Part # (none) -> C21189; Manufacturer (none) -> UNI-ROYAL(Uniroyal Elec); Manufacturer Part (none) -> 0603WAF0000T5E; Supplier Part (none) -> C21189
- R70: LCSC Part # C17168 -> C17477; MPN ERJ-6GEY0R00V -> 0805W8F0000T5E; Manufacturer Panasonic Industry -> UNI-ROYAL(Uniroyal Elec); Manufacturer Part ERJ-6GEY0R00V -> 0805W8F0000T5E; Supplier Part (none) -> C17477
- R71: LCSC Part # (none) -> C25900; Manufacturer (none) -> UNI-ROYAL(Uniroyal Elec); Manufacturer Part (none) -> 0402WGF4701TCE; Supplier Part (none) -> C25900
- TP1: value max +15V! -> +15V!
- TP8: value SP OUT -> SP+; now not fitted
- TP9: value SP OUT -> SP-; now not fitted
- U13: LCSC Part # (none) -> C478472; Manufacturer (none) -> Texas Instruments; Manufacturer Part (none) -> TAS5805MPWPR; Supplier Part (none) -> C478472
Connections:
- net at C91.1, L12.1, U13.20 (OUT_B-): now also C89.1, U13.17 (OUT_B+); no longer C90.1, U13.23 (OUT_A-)
- net at C88.1, L11.1, U13.26 (OUT_A+): now also C90.1, U13.23 (OUT_A-); no longer C89.1, U13.17 (OUT_B+)
Other:
- moved on the sheet: C100, C101, J5, L11, L12
