File: leds.kicad_sch (KiCad schematic)
At the start: 12 parts

Commit message: Publish KiCad 10 hardware updates
Refresh the Nest Mini v2 drop-in PCB project in KiCad 10 and publish the accumulated schematic and board updates as a single clean mainline change.

Remove the unused USB-C power/input branch from the power sheet, including the USB connector path, data switching, VBUS switching, and associated support parts, while preserving the pogo-accessible USB signals where needed. Add the ESP32-C6 1x05 pogo connector with the J2-style pin order for GND, boot, reset, USB D-, and USB D+ without a 3.3 V pin.

Add a 5 V SN74AHCT1G125 buffer for the LED data input, with local decoupling and a 47 ohm series output resistor, so the LED chain receives a buffered LED_WS2812_5V signal from the ESP_WS2812 control net.

Carry forward the KiCad 10 project save state and schematic cleanups for the XMOS, ESP32, audio, LED, and power sheets without changing the TAS amplifier topology.
Parts:
- added C112: 100nF, Capacitor_SMD:C_0402_1005Metric, symbol Device:C
- added R73: 47R, Resistor_SMD:R_0402_1005Metric, symbol Device:R
- added U14: SN74AHCT1G125DBVR, Package_TO_SOT_SMD:SOT-23-5, symbol 74xGxx:74AHCT1G125
- renumbered C92 to C106, C93 to C107, C94 to C108, C95 to C109, C96 to C110, C97 to C111
Connections:
- net +5V: now also C112.1, U14.5 (VCC)
- net ESP_WS2812: now also U14.2; no longer LED1.3 (DIN)
- net GND: now also C112.2, U14.1, U14.3 (GND)
- new net: R73.1, U14.4
- new net LED_WS2812_5V: LED1.3 (DIN), R73.2
