File: leds.kicad_sch (KiCad schematic)
At the start: 15 parts, among them U14 SN74AHCT1G125DBVR

Commit message: v3 hardware ready for prototyping
Parts:
- C106, C107, C108, C109, C110, C111, C112: Dielectric X5R -> X7R; Manufacturer (none) -> Samsung Electro-Mechanics; Manufacturer Part (none) -> CL05B104KO5NNNC
- R73: value 47R -> 33R; LCSC Part # (none) -> C25105; Manufacturer (none) -> UNI-ROYAL(Uniroyal Elec); Manufacturer Part (none) -> 0402WGF330JTCE; Supplier Part (none) -> C25105; Tolerance 5% -> 1%
- U14: LCSC Part # (none) -> C7484; Supplier Part (none) -> C7484
