File: esp32c6fh8_sch.kicad_sch (KiCad schematic)
At the start: 29 parts, among them U16 ESP32-C6FH8, Y2 40MHz

Commit message: Publish KiCad 10 hardware updates
Refresh the Nest Mini v2 drop-in PCB project in KiCad 10 and publish the accumulated schematic and board updates as a single clean mainline change.

Remove the unused USB-C power/input branch from the power sheet, including the USB connector path, data switching, VBUS switching, and associated support parts, while preserving the pogo-accessible USB signals where needed. Add the ESP32-C6 1x05 pogo connector with the J2-style pin order for GND, boot, reset, USB D-, and USB D+ without a 3.3 V pin.

Add a 5 V SN74AHCT1G125 buffer for the LED data input, with local decoupling and a 47 ohm series output resistor, so the LED chain receives a buffered LED_WS2812_5V signal from the ESP_WS2812 control net.

Carry forward the KiCad 10 project save state and schematic cleanups for the XMOS, ESP32, audio, LED, and power sheets without changing the TAS amplifier topology.
Parts:
- added J2: C6 PROGRAM POGO, Connector_PinHeader_2.54mm:PinHeader_1x05_P2.54mm_Vertical, symbol Connector_Generic:Conn_01x05
- C44: renamed from C104; now not fitted
- R32: renamed from R75; now not fitted
- renumbered C103 to C40, C115 to C41, C102 to C42, C101 to C43, C107 to C45, C108 to C46, C114 to C47, C109 to C48, C113 to C49, C110 to C50, C111 to C51, C112 to C52, C105 to C53, C106 to C54, C100 to C55, D7 to D2, FB6 to FB2, L8 to L10, L10 to L7, L11 to L8, R74 to R31, R76 to R33, R77 to R34, U16 to U8
Connections:
- net C6_USB_N: now also J2.4 (Pin_4)
- net C6_USB_P: now also J2.5 (Pin_5)
- net ESP_C6_GPIO9: now also J2.2 (Pin_2)
- net ESP_C6_RST: now also J2.3 (Pin_3)
- net GND: now also J2.1 (Pin_1)
- net ESP_C6_BOOT: no longer names the net of C44.1, R32.2
- net ESP_C6_BOOT: no longer U8.6 (GPIO0/XTAL_32K_P)
- no-connect marks 15 -> 16

Commit message: Publish ESP32-P4 multi-sheet hardware redesign
Parts:
- removed C44: 12pF, Capacitor_SMD:C_0402_1005Metric, symbol Device:C
- removed R32: 10k, Resistor_SMD:R_0402_1005Metric, symbol Device:R
- AE2, C40, C41, C42, C43, C45, C46, C47, C48, C49, C50, C51, C52, C53, C54, C55, D2, FB2, L10, L8, L9, R31, R33, R34, Y2: Function ESP32 -> ESP32-C6
- J2, U8: Function (none) -> ESP32-C6
- L7: Function ESP32C6 -> ESP32-C6
