File: esp32c6.kicad_sch (KiCad schematic)
At the start: 28 parts, among them J2 C6 PROGRAM POGO, U8 ESP32-C6FH8, Y2 40MHz

Commit message: v3 hardware changes
Full redesing, ready for prototype order
Other:
- note added: "JTAG"
- moved on the sheet: C40, C41, D2, FB2, J2, R31

Commit message: v3 hardware ready for prototyping
Parts:
- AE2: Supplier Part (none) -> C89334
- C41: Supplier Part (none) -> C14663
- C42, C43: Supplier Part (none) -> C1547
- C46: Supplier Part (none) -> C48346
- C47, C48, C49, C50, C54: Supplier Part (none) -> C1525
- C51, C53: Supplier Part (none) -> C52923
- C52: Supplier Part (none) -> C15525
- C55: Dielectric X5R -> NP0; Supplier Part (none) -> C327292; Voltage 10V -> 50V
- FB2: Supplier Part (none) -> C14709
- L10: Supplier Part (none) -> C16526
- L7: LCSC Part # (none) -> C341784; Manufacturer (none) -> Murata; Manufacturer Part (none) -> LQW15AN24NJ00D; Supplier Part (none) -> C341784
- L8: Supplier Part (none) -> C162540
- L9: Supplier Part (none) -> C434826
- U8: Manufacturer (none) -> Espressif Systems; Manufacturer Part (none) -> ESP32-C6FH8
- Y2: LCSC Part # C424431 -> C1870451; MPN TAXM40M4ZCBCDT2T -> (none); Manufacturer Yajingxin -> Murata; Manufacturer Part TAXM40M4ZCBCDT2T -> XRCGB40M000F1S1BR0; Supplier Part (none) -> C1870451
