File: esp32s3.kicad_sch (KiCad schematic)
At the start: 40 parts, among them J1 Conn_01x05, U5 ESP32-S3R8, U6 W25Q128JVSIQ, U7 MPR121QR2, Y1 40MHz

Commit message: v3 hardware changes
Full redesing, ready for prototype order
Parts:
- C35: value 1uF -> 100nF; Dielectric X5R -> X7R; LCSC Part # C52923 -> (none); MPN CL05A105KA5NQNC -> CL05B104KO5NNNC; Manufacturer Part CL05A105KA5NQNC -> (none); Voltage 25V -> 16V
- R29: value 200k -> 75k; LCSC Part # C25764 -> (none); MPN 0402WGF2003TCE -> 0402WGF7502TCE
Connections:
- net P4_UA0RXD: now reaches U5.23 (GPIO17)
- net P4_BOOT: now reaches U5.45 (MTDO)
- net P4_RST: now reaches U5.47 (MTDI)
- net P4_UA0TXD: now reaches U5.9 (GPIO4)
- net ESP_3V3 renamed S3_3V3
- net I2S_MCLK: no longer names the net of U5.14 (GPIO9)
- no-connect marks 18 -> 15
Other:
- moved on the sheet: AE1, C20, C21, C22, C23, C24, C25, C26, C27, C28, C29, C30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

Commit message: v3 hardware ready for prototyping
Parts:
- added L13: 24nH, Inductor_SMD:L_0402_1005Metric, symbol Device:L
- AE1: Supplier Part (none) -> C89334
- C21: Supplier Part (none) -> C14663
- C22, C23: Supplier Part (none) -> C1547
- C24: Dielectric X5R -> NP0; Supplier Part (none) -> C327292; Voltage 10V -> 50V
- C26, C27, C29, C30, C31, C34, C36, C37: Supplier Part (none) -> C1525
- C28, C32, C38: Supplier Part (none) -> C52923
- C33: Supplier Part (none) -> C48346
- C35: LCSC Part # (none) -> C1525; Manufacturer Part (none) -> CL05B104KO5NNNC; Supplier Part (none) -> C1525
- C39: Supplier Part (none) -> C15525
- FB1: Supplier Part (none) -> C14709
- L4: Supplier Part (none) -> C16526
- L5: Supplier Part (none) -> C434826
- L6: Supplier Part (none) -> C162540
- R18, R19: Supplier Part (none) -> C25900; Tolerance 5% -> 1%
- R29: LCSC Part # (none) -> C2909383; MPN 0402WGF7502TCE -> FRC0402F7502TS; Manufacturer UNI-ROYAL(Uniroyal Elec) -> FOJAN; Manufacturer Part (none) -> FRC0402F7502TS; Supplier Part (none) -> C2909383
- R30: LCSC Part # C26087 -> C26083; MPN 0402WGJ0105TCE -> (none); Manufacturer Part (none) -> 0402WGF1004TCE; Supplier Part (none) -> C26083
- U5: Supplier Part (none) -> C2913194
- U6: Supplier Part (none) -> C97521
- U7: Manufacturer Part (none) -> MPR121QR2; Supplier Part (none) -> C91322
- Y1: LCSC Part # C424431 -> C1870451; MPN TAXM40M4ZCBCDT2T -> (none); Manufacturer Yajingxin -> Murata; Manufacturer Part TAXM40M4ZCBCDT2T -> XRCGB40M000F1S1BR0; Supplier Part (none) -> C1870451
Connections:
- net at C22.2, Y1.3: now also L13.1; no longer U5.54 (XTAL_P)
- new net: L13.2, U5.54 (XTAL_P)
