File: esp32p4.kicad_sch (KiCad schematic)
At the start: 75 parts, among them J3 P4 PROGRAM POGO, Q3 BC847B, U11 SN74LVC125APWR, U12 TLV73333PDBVR, U9 W25Q128JVSIQ, Y3 40MHz

Commit message: v3 hardware changes
Full redesing, ready for prototype order
Parts:
- removed C59: 12pF, Capacitor_SMD:C_0402_1005Metric, symbol Device:C
- removed C72: 100nF, Capacitor_SMD:C_0402_1005Metric, symbol Device:C
- added C60: 100nF, Capacitor_SMD:C_0603_1608Metric, symbol Device:C
- added FB3: 120R, Onju:BLM18PG121SN1D, symbol Device:FerriteBead
- added R37: 10k, Resistor_SMD:R_0402_1005Metric, symbol Device:R
- added R69: 100k, Resistor_SMD:R_0402_1005Metric, symbol Device:R
- R58: value 1k -> 10k; LCSC Part # C11702 -> (none); Manufacturer Part 0402WGF1001TCE -> (none); Supplier Part C11702 -> (none)
Connections:
- net VDDIO is gone; now on net P4_3V3: C84.1, R58.2, U11.14 (VCC)
- net +3V3: now also FB3.1
- net GND: now also C60.2, R69.1
- net MIC_CLK: now also U4.10 (GPIO9), R69.2
- net MIC_CLK_M: no longer U4.10 (GPIO9)
- net MIC_DATA_1: now also U4.11 (GPIO10)
- net MIC_DATA_2: now also U4.12 (GPIO11)
- net MIC_DATA_M_1: no longer U4.11 (GPIO10)
- net MIC_DATA_M_2: no longer U4.12 (GPIO11)
- net P4_BOOT: now also U4.66 (GPIO35); no longer U4.104 (GPIO0)
- net P4_USB_N: now also U4.52 (GPIO24/USB1P1_N0); no longer U4.49 (USB-DM)
- net P4_USB_P: now also U4.53 (GPIO25/USB1P1_P0); no longer U4.50 (USB-DP)
- net at U4.68 (GPIO36): now also R37.2
- net P4_UA0TXD: now reaches U4.69 (GPIO37)
- net P4_UA0RXD: now reaches U4.70 (GPIO38)
- net ESP_3V3 renamed P4_3V3
- net P4_3V3: now also C60.1, FB3.2, R37.1; no longer R59.2
- new net S3_3V3: R59.2
- no-connect marks 55 -> 56
Other:
- note added: "JTAG"
- moved on the sheet: C113, C114, C115, C116, C117, C118, C119, C120, C121, C122, C123, C124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

Commit message: v3 hardware ready for prototyping
Parts:
- C120, C128, C136, C138: LCSC Part # (none) -> C19702; Manufacturer Part (none) -> CL10A106KP8NNNC; Supplier Part (none) -> C19702; Voltage 25V -> 10V
- C133: LCSC Part # (none) -> C15195; Manufacturer Part (none) -> CL05B103KB5NNNC; Supplier Part (none) -> C15195; Voltage 16V -> 50V
- C44: Supplier Part (none) -> C1525
- C56, C57: Supplier Part (none) -> C1547
- C58: LCSC Part # C52923 -> C15849; Manufacturer Part CL05A105KA5NQNC -> CL10A105KB8NNNC; Supplier Part (none) -> C15849; Voltage 25V -> 50V
- C60: Supplier Part (none) -> C14663
- C78: Dielectric X7R -> X5R; LCSC Part # C86018 -> C23630; Manufacturer Murata Electronics -> Samsung Electro-Mechanics; Manufacturer Part GRM188R71A225KE15D -> CL10A225KO8NNNC; Supplier Part C86018 -> C23630; Voltage 10V -> 16V
- C9: LCSC Part # (none) -> C19666; Manufacturer Part (none) -> CL10A475KO8NNNC; Supplier Part (none) -> C19666; Voltage 25V -> 16V
- D3: MANUFACTURER ON SEMICONDUCTOR -> DOWO; MP RB521S30T1G -> RB521S30T1G-DW; Manufacturer ON SEMICONDUCTOR -> DOWO; Manufacturer Part RB521S30T1G -> RB521S30T1G-DW
- FB3: Supplier Part (none) -> C14709
- J3: Function ESP32-C6 -> ESP32-P4
- MK1, MK2, MK3: MP T3902 -> MMICT390200012
- Q3: value BC847B -> MMBT3904; symbol Transistor_BJT:Q_NPN_BCE -> Transistor_BJT:Q_NPN_BEC; LCSC Part # C20069135 -> C20526; MANUFACTURER hongjiacheng -> CJ(Jiangsu Changjing Electronics Technology Co., Ltd.); MP BC847B -> MMBT3904; Manufacturer hongjiacheng -> CJ(Jiangsu Changjing Electronics Technology Co., Ltd.); Manufacturer Part BC847B -> MMBT3904; Supplier Part C20069135 -> C20526
- R36: Function (none) -> ESP32-P4; Supplier Part (none) -> C17168
- R52, R53, R56, R60, R61, R62, R63, R64, R65, R66: Tolerance 5% -> 1%
- R58: LCSC Part # (none) -> C25744; Manufacturer Part (none) -> 0402WGF1002TCE; Supplier Part (none) -> C25744; Tolerance 5% -> 1%
- R69: LCSC Part # (none) -> C25741; Manufacturer Part (none) -> 0402WGF1003TCE; Supplier Part (none) -> C25741
- U4: value (none) -> ESP32-P4NRW32X; LCSC Part # (none) -> C54540373; Manufacturer (none) -> Espressif Systems; Manufacturer Part (none) -> ESP32-P4NRW32X; Supplier Part (none) -> C54540373
- U9: Supplier Part (none) -> C97521
- Y3: LCSC Part # C424431 -> C1870451; MPN TAXM40M4ZCBCDT2T -> (none); Manufacturer Yajingxin -> Murata; Manufacturer Part TAXM40M4ZCBCDT2T -> XRCGB40M000F1S1BR0; Supplier Part (none) -> C1870451
Connections:
- net GND: now also Q3.2 (E); no longer Q3.3 (E)
- net at R55.1, U12.3 (EN): now also Q3.3 (C); no longer Q3.2 (C)

Commit message: v3 hardware ready for prototyping
Parts:
- R54: value 3.3k -> 100k; LCSC Part # C25890 -> C25741; Manufacturer Part 0402WGF3301TCE -> 0402WGF1003TCE; Supplier Part C25890 -> C25741
Connections:
- net VDD_MIC: no longer C85.1, C86.1, C87.1
- net at MK1.2 (SELECT), MK1.5 (VDD), R63.2: now also C86.1
- net at MK2.5 (VDD), R64.2: now also C85.1
- net at MK3.2 (SELECT), MK3.5 (VDD), R65.2: now also C87.1
Other:
- moved on the sheet: R60, R61, R62
