File: power_handling.kicad_sch (KiCad schematic)
At the start: 36 parts, among them U1 TLV62569DRLR, U2 TPS62130, U3 TPS62130

Commit message: v3 hardware ready for prototyping
Parts:
- L1, L2, L3: footprint Inductor_SMD:L_Cenker_CKCS4020 -> Onju:IND_SRP4020TA-2R2M
Changed lines of the file:
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@@
 			)
 		)
-		(property "Footprint" "Inductor_SMD:L_Cenker_CKCS4020"
+		(property "Footprint" "Onju:IND_SRP4020TA-2R2M"
 			(at 199.39 95.25 0)
 			(hide yes)
@@
 			)
 		)
-		(property "Footprint" "Inductor_SMD:L_Cenker_CKCS4020"
+		(property "Footprint" "Onju:IND_SRP4020TA-2R2M"
 			(at 69.85 97.79 0)
 			(hide yes)
@@
 			)
 		)
-		(property "Footprint" "Inductor_SMD:L_Cenker_CKCS4020"
+		(property "Footprint" "Onju:IND_SRP4020TA-2R2M"
 			(at 208.28 35.56 0)
 			(hide yes)
